Commit message: Added camera sensor-

File: shooting_set_description/urdf/shooting_set.xacro (robot description, xacro)
@@ -361,4 +361,6 @@
    -->
 </link>
+<link name="${robot_name}_camera_link_1">
+</link>
 <link name="base_footprint">
 </link>
@@ -367,4 +369,9 @@
   <parent link="${robot_name}_base_link"/>
   <child link="base_footprint"/>
+</joint>
+<joint name="${robot_name}_camera_base_joint" type="fixed">
+  <origin xyz="0.0 0.0 0.02" rpy="0 0 0"/>
+  <parent link="${robot_name}_base_link"/>
+  <child link="${robot_name}_camera_link_1"/>
 </joint>
 <joint name="${robot_name}_lidar_base_joint" type="fixed">
@@ -477,3 +484,4 @@
 <xacro:mechanum_drive fl="${robot_name}_lf_wheel_joint" fr="${robot_name}_rf_wheel_joint" bl="${robot_name}_lb_wheel_joint" br="${robot_name}_rb_wheel_joint" radius="0.05" />
 <xacro:lidar frame_id="${robot_name}_lidar_link_1" topic="${robot_name}_scan"/>
+<xacro:camera frame_id="${robot_name}_camera_link_1" topic="${robot_name}_camera" height="400" width="500"/>
 </robot>
