Commit message: added lidar in both robot

File: rbcon_sim/xacro/gazebo.xacro (robot description, xacro)
@@ -21,5 +21,5 @@
     <xacro:macro name="lidar" params="frame_id topic">
         <gazebo reference="${frame_id}">
-            <sensor name="lidar_sensor" type="gpu_lidar">
+            <sensor name="${frame_id}" type="gpu_lidar">
                 <pose>0 0 0 0 0 0</pose>
                 <gz_frame_id>${frame_id}</gz_frame_id>
@@ -96,5 +96,6 @@
         <plugin filename="libignition-gazebo6-odometry-publisher-system.so"
             name="ignition::gazebo::systems::OdometryPublisher">
-            <odom_frame>${robot_name}_odom</odom_frame>
+            <!-- <odom_frame>${robot_name}_odom</odom_frame> -->
+            <odom_frame>odom</odom_frame>
             <robot_base_frame>${robot_name}_base_link</robot_base_frame>
             <odom_topic>/${robot_name}_odom</odom_topic>
@@ -102,10 +103,9 @@
         </plugin>
         <plugin filename="libignition-gazebo6-imu-system.so" name="ignition::gazebo::systems::Imu" />
-        <!-- <plugin filename="libignition-sensors-lidar.so"
-        name="ignition::gazebo::sensors::Lidar"/> -->
-        <plugin filename="libignition-gazebo-sensors-system.so"
+        <!-- <plugin filename="libignition-sensors6-gpu_lidar.so" name="ignition::gazebo::sensors::Lidar"/> -->
+        <!-- <plugin filename="libignition-gazebo-sensors-system.so"
             name="ignition::gazebo::systems::Sensors">
             <render_engine>ogre</render_engine>
-        </plugin>
+        </plugin> -->
         <!-- <plugin filename="libignition-gazebo6-velocity-control-system.so.6"
             name="ignition::gazebo::systems::VelocityControl">

File: shooting_set_description/urdf/shooting_set.xacro (robot description, xacro)
@@ -351,4 +351,19 @@
   </collision>
 </link>
+<link name="${robot_name}_lidar_link_1">
+  <!-- <visual>
+    <origin xyz="0 0 0.1" rpy="0 0 0"/>
+    <geometry>
+      <cylinder length="0.02" radius="0.05"/>
+    </geometry>
+    <material name="black"/>
+  </visual>
+   -->
+</link>
+<joint name="${robot_name}_lidar_base_joint" type="fixed">
+  <origin xyz="0.0 0.0 0.02" rpy="0 0 0"/>
+  <parent link="${robot_name}_base_link"/>
+  <child link="${robot_name}_lidar_link_1"/>
+</joint>
 <joint name="${robot_name}_lb_wheel_joint" type="continuous">
   <origin xyz="-0.175 0.26 0.025" rpy="0 0 0"/>
@@ -454,3 +469,4 @@
 </joint> -->
 <xacro:mechanum_drive fl="${robot_name}_lf_wheel_joint" fr="${robot_name}_rf_wheel_joint" bl="${robot_name}_lb_wheel_joint" br="${robot_name}_rb_wheel_joint" radius="0.05" />
+<xacro:lidar frame_id="${robot_name}_lidar_link_1" topic="${robot_name}_scan"/>
 </robot>

Commit message: feature added localization-

File: rbcon_sim/xacro/gazebo.xacro (robot description, xacro)
@@ -96,6 +96,6 @@
         <plugin filename="libignition-gazebo6-odometry-publisher-system.so"
             name="ignition::gazebo::systems::OdometryPublisher">
-            <!-- <odom_frame>${robot_name}_odom</odom_frame> -->
-            <odom_frame>odom</odom_frame>
+            <odom_frame>${robot_name}_odom</odom_frame>
+            <!-- <odom_frame>odom</odom_frame> -->
             <robot_base_frame>${robot_name}_base_link</robot_base_frame>
             <odom_topic>/${robot_name}_odom</odom_topic>

File: shooting_set_description/urdf/shooting_set.xacro (robot description, xacro)
@@ -361,4 +361,11 @@
    -->
 </link>
+<link name="base_footprint">
+</link>
+<joint name="${robot_name}_footprint_base_joint" type="fixed">
+  <origin xyz="0.0 0.0 0.02" rpy="0 0 0"/>
+  <parent link="${robot_name}_base_link"/>
+  <child link="base_footprint"/>
+</joint>
 <joint name="${robot_name}_lidar_base_joint" type="fixed">
   <origin xyz="0.0 0.0 0.02" rpy="0 0 0"/>

Commit message: intial commit (FPS) to be check

File: rbcon_sim/xacro/gazebo.xacro (robot description, xacro)
@@ -1,28 +1,31 @@
 <?xml version="1.0" encoding="UTF-8"?>
 <robot xmlns:xacro="http://www.ros.org/wiki/xacro" name="gzbo">
-    <xacro:macro name="mechanum_drive" params="fl fr bl br radius">
+    <!-- Mecanum Drive for Robot 1 -->
+    <xacro:macro name="mechanum_drive" params="robot_name fl fr bl br radius base_frame">
         <gazebo>
             <plugin filename="libignition-gazebo-mecanum-drive-system.so"
                 name="ignition::gazebo::systems::MecanumDrive">
-                <topic>${robot_name}_cmd_vel</topic>
+                <topic>/${robot_name}/cmd_vel</topic>
                 <front_left_joint>${fl}</front_left_joint>
                 <front_right_joint>${fr}</front_right_joint>
                 <back_left_joint>${bl}</back_left_joint>
                 <back_right_joint>${br}</back_right_joint>
-                <!-- odometry topic -->
-                <odom_topic>/${robot_name}_odom</odom_topic>
-                <!-- tf topics and frames -->
+                <!-- Odometry -->
+                <odom_topic>/${robot_name}/odom</odom_topic>
+                <!-- TF -->
+                <!-- <tf_topic>/${robot_name}/tf</tf_topic> -->
                 <tf_topic>/tf</tf_topic>
-                <frame_id>odom</frame_id>
-                <child_frame_id>${robot_name}_base_link</child_frame_id>
+                <frame_id>/${robot_name}/odom</frame_id>
+                <child_frame_id>${base_frame}</child_frame_id>
             </plugin>
         </gazebo>
     </xacro:macro>
-    <xacro:macro name="lidar" params="frame_id topic">
+    <!-- LiDAR Macro -->
+    <xacro:macro name="lidar" params="robot_name frame_id topic">
         <gazebo reference="${frame_id}">
             <sensor name="${frame_id}" type="gpu_lidar">
                 <pose>0 0 0 0 0 0</pose>
                 <gz_frame_id>${frame_id}</gz_frame_id>
-                <topic>${topic}</topic>
+                <topic>/${robot_name}/${topic}</topic>
                 <update_rate>10</update_rate>
                 <ray>
@@ -34,10 +37,4 @@
                             <max_angle>3.14</max_angle>
                         </horizontal>
-                        <vertical>
-                            <samples>1</samples>
-                            <resolution>1</resolution>
-                            <min_angle>0</min_angle>
-                            <max_angle>0</max_angle>
-                        </vertical>
                     </scan>
                     <range>
@@ -77,44 +74,30 @@
         </gazebo>
     </xacro:macro>
-    <xacro:macro name="imu" params="frame_id topic">
-        <gazebo reference="${frame_id}">
-            <sensor type="imu" name="${topic}">
-                <topic>${topic}</topic>
-                <update_rate>30.0</update_rate>
-                <always_on>1</always_on>
-            </sensor>
-            <plugin filename="libignition-gazebo-imu-system.so"
-                name="ignition::gazebo::systems::Imu">
+    <!-- Joint State and Odometry Plugin -->
+    <xacro:macro name="robot_plugins" params="robot_name base_frame">
+        <gazebo>
+            <plugin filename="libignition-gazebo6-joint-state-publisher-system.so"
+                name="ignition::gazebo::systems::JointStatePublisher">
+                <topic>/${robot_name}/joint_states</topic>
             </plugin>
+            <plugin filename="libignition-gazebo6-odometry-publisher-system.so"
+                name="ignition::gazebo::systems::OdometryPublisher">
+                <odom_frame>${robot_name}/odom</odom_frame>
+                <robot_base_frame>${base_frame}</robot_base_frame>
+                <odom_topic>/${robot_name}/odom</odom_topic>
+                <!-- <tf_topic>/${robot_name}/tf</tf_topic> -->
+                <tf_topic>/tf</tf_topic>
+            </plugin>
+            <plugin filename="libignition-gazebo6-imu-system.so"
+                name="ignition::gazebo::systems::Imu" />
         </gazebo>
     </xacro:macro>
-    <gazebo>
-        <plugin filename="libignition-gazebo6-joint-state-publisher-system.so"
-            name="ignition::gazebo::systems::JointStatePublisher">
-            <topic>${robot_name}_joint_states</topic>
-        </plugin>
-        <plugin filename="libignition-gazebo6-odometry-publisher-system.so"
-            name="ignition::gazebo::systems::OdometryPublisher">
-            <odom_frame>${robot_name}_odom</odom_frame>
-            <!-- <odom_frame>odom</odom_frame> -->
-            <robot_base_frame>${robot_name}_base_link</robot_base_frame>
-            <odom_topic>/${robot_name}_odom</odom_topic>
-            <tf_topic>/tf</tf_topic>
-        </plugin>
-        <!-- <plugin
-            filename="ignition-gazebo-joint-controller-system"
-            name="gz::sim::systems::JointController">
-            <joint_name>${robot_name}_joint_control</joint_name>
-            <initial_velocity>5.0</initial_velocity>
-        </plugin> -->
-        <plugin filename="libignition-gazebo6-imu-system.so" name="ignition::gazebo::systems::Imu" />
-        <!-- <plugin filename="libignition-sensors6-gpu_lidar.so" name="ignition::gazebo::sensors::Lidar"/> -->
-        <!-- <plugin filename="libignition-gazebo-sensors-system.so"
-            name="ignition::gazebo::systems::Sensors">
-            <render_engine>ogre</render_engine>
-        </plugin> -->
-        <!-- <plugin filename="libignition-gazebo6-velocity-control-system.so.6"
-            name="ignition::gazebo::systems::VelocityControl">
-        </plugin> -->
-    </gazebo>
+    <!-- Add Robot 1 -->
+    <!-- <xacro:mechanum_drive robot_name="robot1" fl="fl_joint1" fr="fr_joint1" bl="bl_joint1" br="br_joint1" radius="0.1"/>
+    <xacro:lidar robot_name="robot1" frame_id="robot1_lidar" topic="scan"/>
+    <xacro:robot_plugins robot_name="robot1" base_frame="robot1_base_link"/> -->
+    <!-- Add Robot 2 -->
+    <!-- <xacro:mechanum_drive robot_name="robot2" fl="fl_joint2" fr="fr_joint2" bl="bl_joint2" br="br_joint2" radius="0.1"/>
+    <xacro:lidar robot_name="robot2" frame_id="robot2_lidar" topic="scan"/>
+    <xacro:robot_plugins robot_name="robot2" base_frame="robot2_base_link"/> -->
 </robot>

File: rbcon_sim/xacro/ros2_control.xacro (robot description, xacro)
@@ -1,14 +1,31 @@
 <?xml version="1.0"?>
 <robot xmlns:xacro="http://www.ros.org/wiki/xacro" name="ros2_control">
+    <!-- Define ros2_control hardware interface -->
+    <!-- <ros2_control name="ros2_control" type="system">
+        <hardware>
+            <plugin>ign_ros2_control/IgnitionSystemInterface</plugin>
+        </hardware>
+        <joint name="joint1">
+            <command_interface name="position"/>
+            <state_interface name="position"/>
+            <state_interface name="velocity"/>
+        </joint>
+        <joint name="joint2">
+            <command_interface name="position"/>
+            <state_interface name="position"/>
+            <state_interface name="velocity"/>
+        </joint>
+    </ros2_control> -->
+    <!-- Load ROS2 Control plugin -->
     <gazebo>
-    <plugin filename="ign_ros2_control-system" name="ign_ros2_control::IgnitionROS2ControlPlugin">
-        <robot_param>robot_description</robot_param>
-        <robot_param_node>robot_state_publisher</robot_param_node>
-        <!-- <parameters>$(find ign_ros2_control_demos)/config/cart_controller.yaml</parameters> -->
-    </plugin>
+        <plugin filename="ign_ros2_control-system" name="ign_ros2_control::IgnitionROS2ControlPlugin">
+            <robot_param>robot_description</robot_param>
+            <robot_param_node>robot_state_publisher</robot_param_node>
+        </plugin>
     </gazebo>
+    <!-- Load Joint Trajectory Controller -->
     <gazebo>
-    <plugin filename="libignition-gazebo6-joint-trajectory-controller-system.so.6" name="ignition::gazebo::systems::JointTrajectoryController">
-    </plugin>
+        <plugin filename="libignition-gazebo6-joint-trajectory-controller-system.so.6"
+                name="ignition::gazebo::systems::JointTrajectoryController"/>
     </gazebo>
 </robot>

Commit message: fix slam and localization(Need solve filter dropping issue with lidar link)

File: rbcon_sim/xacro/gazebo.xacro (robot description, xacro)
@@ -43,5 +43,5 @@
                     <range>
                         <min>0.5</min>
-                        <max>10.0</max>
+                        <max>25.0</max>
                         <resolution>0.01</resolution>
                     </range>

File: shooting_set_description/urdf/shooting_set.xacro (robot description, xacro)
@@ -363,10 +363,10 @@
 <link name="${robot_name}_camera_link_1">
 </link>
-<link name="base_footprint">
+<link name="${robot_name}_base_footprint">
 </link>
 <joint name="${robot_name}_footprint_base_joint" type="fixed">
   <origin xyz="0.0 0.0 0.02" rpy="0 0 0"/>
   <parent link="${robot_name}_base_link"/>
-  <child link="base_footprint"/>
+  <child link="${robot_name}_base_footprint"/>
 </joint>
 <joint name="${robot_name}_camera_base_joint" type="fixed">

Commit message: added omni chassis and velocity effort control

File: rbcon_sim/xacro/gazebo.xacro (robot description, xacro)
@@ -97,9 +97,62 @@
             name="ignition::gazebo::systems::OdometryPublisher">
             <odom_frame>${robot_name}_odom</odom_frame>
-            <!-- <odom_frame>odom</odom_frame> -->
             <robot_base_frame>${robot_name}_base_link</robot_base_frame>
             <odom_topic>/${robot_name}_odom</odom_topic>
             <tf_topic>/tf</tf_topic>
         </plugin>
+        <!-- <plugin filename="libignition-gazebo6-joint-controller-system.so"
+            name="ignition::gazebo::systems::JointController">
+            <joint_name>${robot_name}_upper_shaft_joint</joint_name>
+            <joint_name>${robot_name}_bottom_shaft_joint</joint_name>
+            <joint_name>${robot_name}_frame_joint</joint_name>
+            <initial_velocity>0.5</initial_velocity>
+        </plugin> -->
+        <plugin
+            filename="libignition-gazebo-joint-trajectory-controller-system.so"
+            name="ignition::gazebo::systems::JointTrajectoryController">
+            <topic>${robot_name}_joint_control</topic>
+        </plugin>
+        <!-- <plugin
+            filename="libignition-gazebo-joint-trajectory-controller-system.so"
+            name="ignition::gazebo::systems::JointTrajectoryController">
+            <joint_name>${robot_name}_upper_shaft_joint</joint_name>
+            <velocity_p_gain>0.1</velocity_p_gain>
+            <velocity_i_gain>175</velocity_i_gain>
+            <velocity_cmd_min>-10</velocity_cmd_min>
+            <velocity_cmd_max>10</velocity_cmd_max>
+            <joint_name>${robot_name}_bottom_shaft_joint</joint_name>
+            <velocity_p_gain>0.1</velocity_p_gain>
+            <velocity_i_gain>200</velocity_i_gain>
+            <velocity_cmd_min>-5</velocity_cmd_min>
+            <velocity_cmd_max>5</velocity_cmd_max>
+        </plugin> -->
+        <!-- <plugin
+            filename="libignition-gazebo-joint-trajectory-controller-system.so"
+            name="ignition::gazebo::systems::JointTrajectoryController">
+            <joint_name>${robot_name}_upper_shaft_joint</joint_name>
+            <velocity_p_gain>0.5</velocity_p_gain>
+            <velocity_i_gain>5.0</velocity_i_gain>
+            <velocity_d_gain>0.1</velocity_d_gain>
+            <velocity_i_min>-1</velocity_i_min>
+            <velocity_i_max>1</velocity_i_max>
+            <velocity_cmd_min>-5</velocity_cmd_min>
+            <velocity_cmd_max>5</velocity_cmd_max>
+            <joint_name>${robot_name}_bottom_shaft_joint</joint_name>
+            <velocity_p_gain>0.5</velocity_p_gain>
+            <velocity_i_gain>5.0</velocity_i_gain>
+            <velocity_d_gain>0.1</velocity_d_gain>
+            <velocity_i_min>-1</velocity_i_min>
+            <velocity_i_max>1</velocity_i_max>
+            <velocity_cmd_min>-5</velocity_cmd_min>
+            <velocity_cmd_max>5</velocity_cmd_max>
+        </plugin> -->
+        <!-- <plugin
+            filename="libignition-gazebo-joint-trajectory-controller-system.so"
+            name="ignition::gazebo::systems::JointTrajectoryController">
+            <velocity_p_gain>0.1</velocity_p_gain>
+            <velocity_i_gain>180</velocity_i_gain>
+            <velocity_cmd_min>-10</velocity_cmd_min>
+            <velocity_cmd_max>10</velocity_cmd_max>
+        </plugin> -->
         <!-- <plugin
             filename="ignition-gazebo-joint-controller-system"
@@ -109,12 +162,4 @@
         </plugin> -->
         <plugin filename="libignition-gazebo6-imu-system.so" name="ignition::gazebo::systems::Imu" />
-        <!-- <plugin filename="libignition-sensors6-gpu_lidar.so" name="ignition::gazebo::sensors::Lidar"/> -->
-        <!-- <plugin filename="libignition-gazebo-sensors-system.so"
-            name="ignition::gazebo::systems::Sensors">
-            <render_engine>ogre</render_engine>
-        </plugin> -->
-        <!-- <plugin filename="libignition-gazebo6-velocity-control-system.so.6"
-            name="ignition::gazebo::systems::VelocityControl">
-        </plugin> -->
     </gazebo>
 </robot>

File: shooting_set_description/urdf/shooting_set.xacro (robot description, xacro)
@@ -404,4 +404,5 @@
   <axis xyz="0.0 1.0 0.0"/>
 </joint>
+<!--
 <joint name="${robot_name}_frame_joint" type="fixed">
   <origin xyz="0.25 0.0 0.05" rpy="0 -0.5 0"/>
@@ -409,4 +410,21 @@
   <child link="${robot_name}_frame_1"/>
   <axis xyz="0.0 1.0 0.0"/>
+</joint> -->
+<!-- <joint name="${robot_name}_frame_joint" type="revolute">
+  <origin xyz="0.25 0.0 0.05" rpy="0 -0.5 0"/>
+  <parent link="${robot_name}_base_link"/>
+  <child link="${robot_name}_frame_1"/>
+  <axis xyz="0.0 1.0 0.0"/>
+  <limit effort="10.0" velocity="1.0" lower="-1.57" upper="1.57"/>
+  <dynamics damping="0.5" friction="0.1"/>
+</joint> -->
+<joint name="${robot_name}_frame_joint" type="revolute">
+  <origin xyz="0.25 0.0 0.05" rpy="0 -0.5 0"/>
+  <parent link="${robot_name}_base_link"/>
+  <child link="${robot_name}_frame_1"/>
+  <axis xyz="0.0 1.0 0.0"/>
+  <dynamics damping="0.3"/>
+  <!-- Limits for safety -->
+  <limit effort="75.0" velocity="7.0" lower="-3.14" upper="3.14"/>
 </joint>
 <joint name="${robot_name}_r1" type="continuous">
@@ -482,4 +500,19 @@
    <child link="${robot_name}_base_link"/>
 </joint> -->
+<!-- <gazebo>
+  <plugin name="gazebo_ros_control" filename="libgazebo_ros_control.so"/>
+</gazebo> -->
+<!-- <transmission name="${robot_name}_frame_joint_trans">
+  <type>transmission_interface/SimpleTransmission</type>
+  <joint name="${robot_name}_frame_joint">
+    <hardwareInterface>hardware_interface/PositionJointInterface</hardwareInterface>
+    <hardwareInterface>hardware_interface/VelocityJointInterface</hardwareInterface>
+    <hardwareInterface>hardware_interface/EffortJointInterface</hardwareInterface>
+  </joint>
+  <actuator name="${robot_name}_frame_motor">
+    <hardwareInterface>hardware_interface/EffortJointInterface</hardwareInterface>
+    <mechanicalReduction>1.0</mechanicalReduction>
+  </actuator>
+</transmission> -->
 <xacro:mechanum_drive fl="${robot_name}_lf_wheel_joint" fr="${robot_name}_rf_wheel_joint" bl="${robot_name}_lb_wheel_joint" br="${robot_name}_rb_wheel_joint" radius="0.05" />
 <xacro:lidar frame_id="${robot_name}_lidar_link_1" topic="${robot_name}_scan"/>
