Commit message: Added Control for both robot with Red-gear -FlyWheel -Base Angle -Drive

File: rbcon_sim/xacro/gazebo.xacro (robot description, xacro)
@@ -21,31 +21,30 @@
     <xacro:macro name="lidar" params="frame_id topic">
         <gazebo reference="${frame_id}">
-            <sensor name="${frame_id}" type="gpu_lidar">
+            <sensor name="${frame_id}_lidar" type="gpu_lidar">
                 <pose>0 0 0 0 0 0</pose>
-                <gz_frame_id>${frame_id}</gz_frame_id>
                 <topic>${topic}</topic>
                 <update_rate>10</update_rate>
-                <ray>
+                <ray>  <!-- Changed from ray to ray element -->
                     <scan>
                         <horizontal>
-                            <samples>640</samples>
+                            <samples>300</samples>
                             <resolution>1</resolution>
-                            <min_angle>-3.14</min_angle>
-                            <max_angle>3.14</max_angle>
+                            <min_angle>-3.14</min_angle>  <!-- -80 degrees -->
+                            <max_angle>3.14</max_angle>   <!-- +80 degrees -->
                         </horizontal>
-                        <vertical>
-                            <samples>1</samples>
+                        <!-- <vertical>
+                            <samples>10</samples>
                             <resolution>1</resolution>
-                            <min_angle>0</min_angle>
-                            <max_angle>0</max_angle>
-                        </vertical>
+                            <min_angle>0.0</min_angle>
+                            <max_angle>0.0</max_angle>
+                        </vertical> -->
                     </scan>
                     <range>
-                        <min>0.05</min>
+                        <min>0.08</min>
                         <max>25.0</max>
                         <resolution>0.01</resolution>
                     </range>
                 </ray>
-                <always_on>1</always_on>
+                <alwaysOn>true</alwaysOn>  <!-- Corrected capitalization -->
                 <visualize>true</visualize>
             </sensor>
@@ -107,4 +106,24 @@
             <tf_topic>/tf</tf_topic>
         </plugin>
+        <plugin name="ignition::gazebo::systems::JointController" filename="libignition-gazebo6-joint-controller-system.so">
+            <joint_name>${robot_name}_upper_shaft_joint</joint_name>
+            <topic>${robot_name}_fly_wheel_up</topic>
+            <control_type>velocity</control_type>
+        </plugin>
+        <plugin name="ignition::gazebo::systems::JointController" filename="libignition-gazebo6-joint-controller-system.so">
+            <joint_name>${robot_name}_bottom_shaft_joint</joint_name>
+            <topic>${robot_name}_fly_wheel_dw</topic>
+            <control_type>velocity</control_type>
+        </plugin>
+        <plugin name="ignition::gazebo::systems::JointController" filename="libignition-gazebo6-joint-controller-system.so">
+            <joint_name>${robot_name}_frame_joint</joint_name>
+            <topic>${robot_name}_angle</topic>
+            <control_type>position</control_type>
+        </plugin>
+        <!-- <plugin name="ignition::gazebo::systems::JointPositionController"
+                filename="libignition-gazebo-joint-position-controller-system.so">
+            <joint_name>${robot_name}_frame_joint</joint_name>
+            <topic>${robot_name}_angle</topic>
+        </plugin> -->
         <!-- <plugin
             filename="ignition-gazebo-joint-controller-system"
@@ -114,5 +133,5 @@
         </plugin> -->
         <plugin filename="libignition-gazebo6-imu-system.so" name="ignition::gazebo::systems::Imu" />
-        <plugin filename="libignition-sensors6-gpu_lidar.so" name="ignition::gazebo::sensors::Lidar"/>
+        <!-- <plugin filename="libignition-sensors6-gpu_lidar.so" name="ignition::gazebo::sensors::Lidar"/> -->
          <!-- <plugin filename="VisualizeLidar" name="Visualize Lidar">
         </plugin> -->

File: shooting_set_description/urdf/shooting_set.xacro (robot description, xacro)
@@ -376,5 +376,5 @@
 </joint>
 <joint name="${robot_name}_lidar_base_joint" type="fixed">
-  <origin xyz="0.0 0.0 0.02" rpy="0 0 0"/>
+  <origin xyz="0.0 0.0 0.2" rpy="0 0 0"/>
   <parent link="${robot_name}_base_link"/>
   <child link="${robot_name}_lidar_link_1"/>
@@ -404,5 +404,6 @@
   <axis xyz="0.0 1.0 0.0"/>
 </joint>
-<joint name="${robot_name}_frame_joint" type="fixed">
+<!-- <joint name="${robot_name}_frame_joint" type="fixed"> -->
+<joint name="${robot_name}_frame_joint" type="continuous">
   <origin xyz="0.25 0.0 0.05" rpy="0 -0.5 0"/>
   <parent link="${robot_name}_base_link"/>
@@ -410,4 +411,13 @@
   <axis xyz="0.0 1.0 0.0"/>
 </joint>
+<!-- <joint name="${robot_name}_frame_joint" type="revolute">
+  <parent link="${robot_name}_base_link"/>
+  <child link="${robot_name}_frame_1"/>
+  <origin xyz="0.25 0.0 0.05" rpy="0 -0.5 0"/>
+  <axis xyz="0 1 0"/>
+  <limit lower="-1.57" upper="1.57" effort="100.0" velocity="1.0"/>
+  <dynamics damping="0.1" friction="0.0"/>
+</joint>
+ -->
 <joint name="${robot_name}_r1" type="continuous">
   <origin xyz="-0.596972 -0.22 0.593067" rpy="0 0 0"/>
